Commit message: 3

File: src/navigation_control/urdf/robot.urdf (robot description, URDF)
Before this commit: robot omni_robot, 6 links, 5 joints
Joints:
- joint laser_joint: origin xyz=0.098 0.065 0.077 rpy=0 0 1.5708 -> xyz=0.098 0.065 0.077 rpy=0 0 3.1416

Commit message: Refactor serial data publisher and wheel odometry node for improved communication and data handling
- Updated serial_data_publisher to subscribe to color tracking results and send data in the Vision_Recv_s protocol format.
- Modified OmniWheelCmd structure to accommodate new data fields including target angle, vertical offset, and tracking validity flag.
- Implemented a timer for continuous data sending at 50Hz.
- Enhanced color tracking data parsing with improved error handling.
- Removed unused IMU yaw velocity calculations in wheel_odometry_node and replaced with more accurate IMU yaw change calculations for pose updates.
- Adjusted URDF dimensions for the robot model.
- Improved compiler warning settings in CMakeLists.txt for better code quality.
- Deleted obsolete test scripts for odometry and serial communication.
- Removed outdated documentation on serial communication testing.

File: src/navigation_control/urdf/robot.urdf (robot description, URDF)
Before this commit: robot omni_robot, 6 links, 5 joints
Links:
- link base_link: geometry collision box size=0.262 0.270 0.050; visual box size=0.340 0.300 0.050
